File: Eagle/CG-490/PowerSwitchV1.brd (EAGLE design)
At the start: 23.2 x 26.7 mm, 33 parts, among them IC1 LM393D, IC2 MIC4420M, Q1 2N3906, Q2 STH240N10F7-6, T1 SFH 309

Commit message: updated board layouts
Parts:
- removed COIL-, GND: WIREPADSMD5-2,5, wirepad:5-2,5
- removed LED1: (no value), led:LED3MM
- added TRIG_LED: (no value), led:LED3MM
- R15: value 1k -> 0.005; device rcl:R0603 -> rcl:R1206
- R16: value 1 -> 2; device rcl:0207/7 -> rcl:M0805
- moved R17 86.7 mm to (24.1, 34.3), turned to 270 degrees
- moved D2 84.2 mm to (17.8, 39.4), turned to 180 degrees
- moved D1 76.5 mm to (11.4, 39.4), turned to 180 degrees
- moved R16 71.6 mm to (22.2, 26.7), turned to 90 degrees
- moved Q2 70.0 mm to (6.35, 31.8), turned to 90 degrees
- moved C3 46.9 mm to (24.8, 12.1)
- moved C4 39.9 mm to (26.0, 8.26)
- moved IC2 26.3 mm to (24.1, 19.1)
- moved R15 21.5 mm to (26.7, 34.3)
- moved JP2 9.53 mm to (2.54, 10.2), turned to 90 degrees
- moved C1 3.18 mm to (20.3, 6.35)
- moved IC1 3.18 mm to (13.3, 12.7)
- moved R13 3.18 mm to (17.8, 11.4)
- moved Q1 3.18 mm to (6.99, 12.1)
- moved LED2 3.18 mm to (19.1, 15.9)
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- renumbered T1 to TRIG-TRANS
Connections:
- removed net N$2: LED2.A, R15.1
- net AGND: now also R15.1, TRIG_LED.K; no longer LED1.K
- net GND: no longer GND.1
- net N$13: now also LED2.A; no longer R15.2
- net N$14: now also R15.2
- net N$9: now also TRIG_LED.A; no longer LED1.A
- net OUT: no longer COIL-.1
Routing:
- net ENABLE: track 29.1 -> 10.5 mm, vias 1 -> 2
- net +12V: track 48.0 -> 63.8 mm, vias 2 -> 1
- net N$4: track 0.00 -> 10.3 mm
- net N$9: track 9.20 -> 13.9 mm
- net N$2: track 4.64 -> 0.00 mm
- net N$15: track 0.00 -> 3.20 mm
- net N$13: track 22.0 -> 24.6 mm, vias 0 -> 2
- net N$10: track 0.00 -> 2.29 mm, vias 0 -> 9
- net N$1: track 17.5 -> 18.2 mm
- added copper zone on layer 16, net AGND
- added copper zone on layer 16, net GND
- added copper zone on layer 1, net N$14
- added copper zone on layer 16, net N$14
- added copper zone on layer 1, net OUT
- added copper zone on layer 16, net OUT
Other:
- board size 23.2 x 26.7 mm -> 30.1 x 43.8 mm

Commit message: finalized schematic/pcb, updated report
Parts:
- removed TRIG_LED: (no value), led:LED3MM
- added C_SENSE: (no value), pinhead:1X02
- added TRIG: (no value), pinhead:1X03
- added TRIG_SEL: (no value), jumper:SJ
- added TX: (no value), led:LED3MM
- moved IC2 1.27 mm to (22.9, 19.1)
- renumbered TRIG-TRANS to RX
Connections:
- removed net GND: C3.2, C4.2
- new net N$2: IC2.2, TRIG.1, TRIG_SEL.2
- net AGND: now also C3.2, C4.2, C_SENSE.1, TRIG.3, TX.K; no longer TRIG_LED.K
- net N$13: now also TRIG.2, TRIG_SEL.1; no longer IC2.2
- net N$14: now also C_SENSE.2
- net N$9: now also TX.A; no longer TRIG_LED.A
Routing:
- net AGND: track 0.00 -> 16.7 mm, vias 13 -> 56
- net N$2: track 0.00 -> 8.74 mm, vias 0 -> 1
- net N$13: track 24.6 -> 30.7 mm
- net N$10: track 2.29 -> 5.08 mm, vias 9 -> 10
- net N$9: track 13.9 -> 15.7 mm
- net N$4: track 10.3 -> 8.67 mm
- net N$3: track 3.29 -> 4.76 mm
- net +12V: track 63.8 -> 63.0 mm
- removed copper zone on layer 16, net GND
Other:
- board text added: "+12V"
- board text added: "AN+"
- board text added: "B"
- board text added: "C"
- board text added: "CAT-"
- board text added: "CG-490 PowerSwitchV1 Thomas Kulin 2020"
- board text added: "COIL"
- board text added: "CUR"
- board text added: "E"
- board text added: "EN"
- board text added: "EXT"
- board text added: "GND"
- board text added: "IC1"
- board text added: "INT"
- board text added: "INT is connected to hardware trigger output EXT is connected to MOSFET driver input"
- board text added: "Maximum pulse duration set by C1 charging through R7"
- board text added: "R12 and R2 set the reference voltage."
- board text added: "Short EN to +12V to prevent triggering"
- board text added: "Short R15 & R17 to disable current monitoring"
- board text added: "Short jumper to select internal hardware triggering."
- board text added: "TRIG"

Commit message: updated board layout
Parts:
- moved LED2 0.95 mm to (18.1, 15.9)
Routing:
- net N$3: track 4.76 -> 6.67 mm
- net N$15: track 3.20 -> 4.61 mm
- net N$13: track 30.7 -> 31.8 mm
- net N$11: track 11.3 -> 12.0 mm
